File: kb.kicad_pcb (KiCad board)
At the start: 2 copper layers, 346 x 103 mm, 194 parts, among them J1 Debug, J2 78171-0004, SW1 SW_Push, SW10 SW_Push, SW11 SW_Push, SW12 SW_Push, SW13 SW_Push, SW14 SW_Push, SW15 SW_Push, SW16 SW_Push, SW17 SW_Push, SW18 SW_Push, SW19 SW_Push, SW2 SW_Push, SW20 SW_Push, SW21 SW_Push, SW22 SW_Push, SW23 SW_Push, SW24 SW_Push, SW25 SW_Push, SW26 SW_Push, SW27 SW_Push, SW28 SW_Push, SW29 SW_Push, SW3 SW_Push, SW30 SW_Push, SW31 SW_Push, SW32 SW_Push, SW33 SW_Push, SW34 SW_Push, SW35 SW_Push, SW36 SW_Push, SW37 SW_Push, SW38 SW_Push, SW39 SW_Push, SW4 SW_Push, SW40 SW_Push, SW41 SW_Push, SW42 SW_Push, SW43 SW_Push, SW44 SW_Push, SW45 SW_Push, SW46 SW_Push, SW47 SW_Push, SW48 SW_Push, SW49 SW_Push, SW5 SW_Push, SW50 SW_Push, SW51 SW_Push, SW52 SW_Push, SW53 SW_Push, SW54 SW_Push, SW55 SW_Push, SW56 SW_Push, SW57 SW_Push, SW58 SW_Push, SW59 SW_Push, SW6 SW_Push, SW60 SW_Push, SW61 SW_Push, SW62 SW_Push, SW63 SW_Push, SW64 SW_Push, SW65 SW_Push, SW66 SW_Push, SW67 SW_Push, SW68 SW_Push, SW69 SW_Push, SW7 SW_Push, SW70 SW_Push, SW71 SW_Push, SW72 SW_Push, SW73 SW_Push, SW76 RotaryEncoder_Switch, SW8 SW_Push, SW9 SW_Push, U1 TLV71333PDQN, U2 STM32F412CEUx, Y1 16MHz

Commit message: more routing work
Parts:
- moved D102 295.8 mm to (50.0, 33.6)
- moved R2 295.8 mm to (52.8, 30.1)
- moved R3 295.8 mm to (53.0, 31.8)
- moved R4 295.8 mm to (53.6, 33.6)
- moved D100 295.8 mm to (50.3, 30.3)
- moved D101 295.8 mm to (50.2, 31.9)
- moved D103 95.5 mm to (51.8, 51.8)
- moved R1 95.5 mm to (54.4, 52.6)
- moved C9 87.0 mm to (60.2, 56.7), turned to 0 degrees
- moved U1 84.9 mm to (60.2, 58.7), turned to 90 degrees
- moved C8 82.7 mm to (60.2, 60.7), turned to 0 degrees
- moved C15 35.1 mm to (348.5, 40.0), turned to 90 degrees
- moved C14 34.4 mm to (348.4, 34.0), turned to -90 degrees
- moved R12 29.3 mm to (350.9, 40.0), turned to 90 degrees
- moved R16 29.0 mm to (349.7, 40.0), turned to -90 degrees
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Routing:
- net /COL15: track 63.9 -> 385.7 mm, vias 0 -> 2
- net /ROW4: track 321.1 -> 375.1 mm, vias 0 -> 1
- net /ROW3: track 327.8 -> 367.2 mm, vias 0 -> 1
- net /ROW0: track 285.8 -> 317.7 mm, vias 0 -> 1
- net /ROW2: track 323.8 -> 347.1 mm, vias 0 -> 1
- net /ROW1: track 323.8 -> 337.3 mm, vias 0 -> 1
- net Net-(R13-Pad2): track 0.00 -> 4.40 mm
- net Net-(R12-Pad2): track 0.00 -> 4.30 mm
- net /SWITCH: track 0.00 -> 4.04 mm
- net +3V3: track 2.23 -> 4.08 mm, vias 0 -> 3
- net GND: track 1.88 -> 3.11 mm, vias 3 -> 5
- net /EC11A: track 0.00 -> 1.22 mm
- net /COL7: track 214.3 -> 215.5 mm
- net /EC11B: track 0.00 -> 1.21 mm

Commit message: backup before encoder fix
Parts:
- removed D101, D102: LED, LED_SMD:LED_0402_1005Metric
- added C16: 10n, Capacitor_SMD:C_0603_1608Metric, B.Cu at (335.4, 8.62)
- added C17: 0u1, Capacitor_SMD:C_0603_1608Metric, B.Cu at (20.5, 21.2)
- added SW74: SW_Push, Button_Switch_SMD:SW_SPST_PTS810, B.Cu at (22.1, 24.1)
- added SW75: SW_Push, Button_Switch_SMD:SW_SPST_PTS810, B.Cu at (22.1, 28.3)
- C1, C10, C13, C14, C15, C3, C4, C5, C6, C7: footprint Capacitor_SMD:C_0402_1005Metric -> Capacitor_SMD:C_0603_1608Metric; moved to B.Cu
- C11, C12, C8, C9, TP1, TP2, U2: moved to B.Cu
- Ce: renamed from C2; footprint Capacitor_SMD:C_0402_1005Metric -> Capacitor_SMD:C_0603_1608Metric; moved to B.Cu
- D74: renamed from D103; moved to B.Cu
- D75: renamed from D100; value LED -> BLUE; moved to B.Cu
- J1: footprint Connector_PinHeader_2.54mm:PinHeader_1x06_P2.54mm_Vertical -> Connector_PinHeader_2.54mm:PinHeader_1x06_P2.54mm_Horizontal; moved to B.Cu
- R1, R11, R12, R13, R14, R15, R16, R2, R5, R6, R7, R8, R9: footprint Resistor_SMD:R_0402_1005Metric -> Resistor_SMD:R_0603_1608Metric; moved to B.Cu
- R10: value 1K -> 10K; footprint Resistor_SMD:R_0402_1005Metric -> Resistor_SMD:R_0603_1608Metric; moved to B.Cu
- R3, R4: value 1K5 -> 10K; footprint Resistor_SMD:R_0402_1005Metric -> Resistor_SMD:R_0603_1608Metric; moved to B.Cu
- SW17, SW30, SW69, SW70: footprint PCM_marbastlib-mx:SW_MX_1u -> PCM_marbastlib-mx:SW_MX_1.5u
- SW33, SW59, SW67: footprint PCM_marbastlib-mx:SW_MX_1u -> PCM_marbastlib-mx:SW_MX_1.75u
- SW63, SW64, SW65: footprint PCM_marbastlib-mx:SW_MX_1u -> PCM_marbastlib-mx:SW_MX_1.25u
- U1: footprint Package_SON:Texas_X2SON-4_1x1mm_P0.65mm -> Package_TO_SOT_SMD:SOT-23-5; moved to B.Cu
- Y1: value 16MHz -> XRCGB16M000FXN20R0; moved to B.Cu
- moved R3 284.9 mm to (337.0, 8.62), turned to -90 degrees
- moved R11 86.3 mm to (25.9, 24.1), turned to 90 degrees
- moved TP2 85.6 mm to (26.4, 21.3), turned to 180 degrees
- moved R10 84.7 mm to (23.6, 21.2), turned to 180 degrees
- moved C11 59.3 mm to (20.0, 36.7), turned to 45 degrees
- moved Y1 58.0 mm to (21.9, 37.9), turned to 45 degrees
- moved R9 56.0 mm to (25.9, 28.3), turned to -90 degrees
- moved C12 54.7 mm to (23.7, 39.1), turned to -135 degrees
- moved TP1 54.3 mm to (26.4, 31.1), turned to 180 degrees
- moved C7 53.6 mm to (27.2, 36.9), turned to 135 degrees
- moved C13 51.9 mm to (23.7, 31.1)
- moved C6 51.3 mm to (26.6, 38.6), turned to 135 degrees
- moved R8 49.6 mm to (28.9, 71.3), turned to -90 degrees
- moved R5 49.5 mm to (21.3, 71.3), turned to -90 degrees
- moved R7 49.4 mm to (26.4, 71.3), turned to -90 degrees
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Connections:
- net /LED1 renamed /LED
- R10 pad 1: /BOOT0 -> Net-(R10-Pad1)
- R10 pad 2: Net-(R10-Pad2) -> /BOOT0
- R11 pad 2: Net-(R10-Pad2) -> Net-(R10-Pad1)
- R14 pad 2: /SWITCH -> Net-(R14-Pad2)
- R3 pad 1: Net-(D101-K) -> /SWITCH
- R3 pad 2: GND -> Net-(R14-Pad2)
- R4 pad 1: Net-(D102-K) -> Net-(R4-Pad1)
- R4 pad 2: GND -> /nRST
- R9 pad 2: /nRST -> Net-(R4-Pad1)
- SW76 pad MP: (no net) -> GND
- SW76 pad S1: /SWITCH -> Net-(R14-Pad2)
- TP1 pad 1: GND -> Net-(R4-Pad1)
- TP2 pad 1: Net-(R10-Pad2) -> Net-(R10-Pad1)
- U1 pad 1: +3V3 -> +5V
- U1 pad 4: +5V -> unconnected-(U1-NC-Pad4)
- U1 pad 5: GND -> +3V3
- U2 pad 14: /COL0 -> /COL15
- U2 pad 3: /LED2 -> unconnected-(U2-PC14-Pad3)
- U2 pad 38: /COL15 -> /COL0
- U2 pad 39: /ROW0 -> /ROW4
- U2 pad 4: /LED3 -> unconnected-(U2-PC15-Pad4)
- U2 pad 40: /ROW1 -> /ROW3
- U2 pad 42: /ROW3 -> /ROW1
- U2 pad 43: /ROW4 -> /ROW0
Routing:
- net +3V3: track 4.08 -> 473.3 mm, vias 3 -> 15
- net /EC11A: track 1.22 -> 346.3 mm
- net /EC11B: track 1.21 -> 342.1 mm
- net /SWITCH: track 4.04 -> 336.4 mm
- net /BOOT0: track 0.00 -> 39.7 mm, vias 0 -> 2
- net /USART2_RX_DEBUG: track 0.00 -> 38.5 mm, vias 0 -> 4
- net GND: track 3.11 -> 41.4 mm, vias 5 -> 24
- net /USART2_TX_DEBUG: track 0.00 -> 38.0 mm, vias 0 -> 4
- net /SWDIO: track 0.00 -> 36.8 mm, vias 0 -> 2
- net /SWCLK: track 0.00 -> 34.9 mm
- net /COL0: track 77.8 -> 100.9 mm
- net /COL7: track 215.5 -> 193.0 mm, vias 2 -> 1
- net /COL15: track 385.7 -> 364.4 mm, vias 2 -> 1
- net +5V: track 0.00 -> 19.9 mm
- net /LED: track 0.00 -> 16.9 mm
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- added copper zone on F.Cu, net GND
Other:
- board size 346 x 103 mm -> 341.8 x 98.8 mm
- board text added: "1.25u"
- board text added: "1.5u"
- board text added: "1.75u"
- board text added: "2.25u"
- board text added: "2u"
- board text added: "3V3"
- board text added: "6.25u"
- board text added: "BOOT0"
- board text added: "CLK"
- board text added: "DBG"
- board text added: "DIO"
- board text added: "Designed by Kalyan Sriram"
- board text added: "GND"
- board text added: "KB65 R1"
- board text added: "PWR"
- board text added: "RST"
- board text added: "URX"
- board text added: "USB"
- board text added: "UTX"
