File: kb.kicad_pcb (KiCad board)
At the start: 2 copper layers, 341.8 x 98.8 mm, 199 parts, among them J1 Debug, J2 78171-0004, SW1 SW_Push, SW10 SW_Push, SW11 SW_Push, SW12 SW_Push, SW13 SW_Push, SW14 SW_Push, SW15 SW_Push, SW16 SW_Push, SW17 SW_Push, SW18 SW_Push, SW19 SW_Push, SW2 SW_Push, SW20 SW_Push, SW21 SW_Push, SW22 SW_Push, SW23 SW_Push, SW24 SW_Push, SW25 SW_Push, SW26 SW_Push, SW27 SW_Push, SW28 SW_Push, SW29 SW_Push, SW3 SW_Push, SW30 SW_Push, SW31 SW_Push, SW32 SW_Push, SW33 SW_Push, SW34 SW_Push, SW35 SW_Push, SW36 SW_Push, SW37 SW_Push, SW38 SW_Push, SW39 SW_Push, SW4 SW_Push, SW40 SW_Push, SW41 SW_Push, SW42 SW_Push, SW43 SW_Push, SW44 SW_Push, SW45 SW_Push, SW46 SW_Push, SW47 SW_Push, SW48 SW_Push, SW49 SW_Push, SW5 SW_Push, SW50 SW_Push, SW51 SW_Push, SW52 SW_Push, SW53 SW_Push, SW54 SW_Push, SW55 SW_Push, SW56 SW_Push, SW57 SW_Push, SW58 SW_Push, SW59 SW_Push, SW6 SW_Push, SW60 SW_Push, SW61 SW_Push, SW62 SW_Push, SW63 SW_Push, SW64 SW_Push, SW65 SW_Push, SW66 SW_Push, SW67 SW_Push, SW68 SW_Push, SW69 SW_Push, SW7 SW_Push, SW70 SW_Push, SW71 SW_Push, SW72 SW_Push, SW73 SW_Push, SW74 SW_Push, SW75 SW_Push, SW76 RotaryEncoder_Switch, SW77 SW_Push, SW78 ROT_SKYLOONG_HS, SW8 SW_Push, SW9 SW_Push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

Commit message: split backspace
Parts:
- removed the REF** at (294.7, 8.96)
- added D77: D, Diode_SMD:D_SOD-123, B.Cu at (309.2, 14.0)
- added SW79: SW_Push, PCM_marbastlib-mx:SW_MX_1u, F.Cu at (304.2, 8.97)
- moved D15 9.53 mm to (290.2, 14.0)
- moved SW15 9.53 mm to (285.2, 8.97)
Connections:
- D30 pad 1: /ROW1 -> /ROW2
- SW45 pad 1: /COL14 -> /COL13
Routing:
- net /COL14: track 364.0 -> 392.2 mm
- net /COL13: track 338.9 -> 366.7 mm
- net /ROW2: track 337.7 -> 359.9 mm, vias 2 -> 4
- net /ROW1: track 350.2 -> 370.3 mm, vias 2 -> 4
- net +3V3: track 465.2 -> 453.4 mm
- net Net-(D77-A): track 0.00 -> 9.45 mm
- net /EC11A: track 346.3 -> 349.2 mm
- net /ROW4: track 379.3 -> 380.9 mm
- net /ROW0: track 368.0 -> 366.8 mm
- net /COL15: track 385.0 -> 386.0 mm
Other:
- outline, holes or cut-outs redrawn
- board text added: "R1 February 2025"
- board text added: "~/superuser"
- board text removed: "2u"
- board text removed: "February 2025"
- board text removed: "KB65 R1"

Commit message: final export of r1
Routing:
- net +3V3: track 453.4 -> 459.0 mm
