File: matrix.kicad_sch (KiCad schematic)
At the start: 158 parts, among them SW1 SW_Push, SW10 SW_Push, SW11 SW_Push, SW12 SW_Push, SW13 SW_Push, SW14 SW_Push, SW15 SW_Push, SW16 SW_Push, SW17 SW_Push, SW18 SW_Push, SW19 SW_Push, SW2 SW_Push, SW20 SW_Push, SW21 SW_Push, SW22 SW_Push, SW23 SW_Push, SW24 SW_Push, SW25 SW_Push, SW26 SW_Push, SW27 SW_Push, SW28 SW_Push, SW29 SW_Push, SW3 SW_Push, SW30 SW_Push, SW31 SW_Push, SW32 SW_Push, SW33 SW_Push, SW34 SW_Push, SW35 SW_Push, SW36 SW_Push, SW37 SW_Push, SW38 SW_Push, SW39 SW_Push, SW4 SW_Push, SW40 SW_Push, SW41 SW_Push, SW42 SW_Push, SW43 SW_Push, SW44 SW_Push, SW45 SW_Push, SW46 SW_Push, SW47 SW_Push, SW48 SW_Push, SW49 SW_Push, SW5 SW_Push, SW50 SW_Push, SW51 SW_Push, SW52 SW_Push, SW53 SW_Push, SW54 SW_Push, SW55 SW_Push, SW56 SW_Push, SW57 SW_Push, SW58 SW_Push, SW59 SW_Push, SW6 SW_Push, SW60 SW_Push, SW61 SW_Push, SW62 SW_Push, SW63 SW_Push, SW64 SW_Push, SW65 SW_Push, SW66 SW_Push, SW67 SW_Push, SW68 SW_Push, SW69 SW_Push, SW7 SW_Push, SW70 SW_Push, SW71 SW_Push, SW72 SW_Push, SW73 SW_Push, SW76 RotaryEncoder_Switch, SW77 SW_Push, SW8 SW_Push, SW9 SW_Push

Commit message: fixed encoder
Parts:
- added SW78: ROT_SKYLOONG_HS, PCM_marbastlib-various:ROT_SKYLOONG_HS-Switch, symbol PCM_marbastlib-various:ROT_SKYLOONG_HS-Switch
Connections:
- net GND: now also R12.2, R16.1, SW76.B, SW78.B, SW78.C; no longer SW76.MP
- net SW77: now reaches D76.2 (A), SW77.2
- net SW77: now also SW76.MP
- net A: now reaches R13.2, R15.1, SW76.A
- net A: now also SW78.A
- net S1: now reaches R14.2, R3.2, SW76.S1
- net S1: now also SW78.S
Other:
- note added: "hack to make pads drill correctly not used electrically"
Changed lines of the file:
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@@
 	)
 	(junction
+		(at 353.06 59.69)
+		(diameter 0)
+		(color 0 0 0 0)
+	)
+	(junction
 		(at 228.6 118.11)
 		(diameter 0)
@@
 	(wire
 		(pts
+			(xy 59.69 267.97) (xy 63.5 267.97)
+		)
+		(stroke
+			(width 0)
+			(type default)
+		)
+	)
+	(wire
+		(pts
 			(xy 279.4 105.41) (xy 281.94 105.41)
 		)
@@
 	(wire
 		(pts
+			(xy 353.06 59.69) (xy 360.68 59.69)
+		)
+		(stroke
+			(width 0)
+			(type default)
+		)
+	)
+	(wire
+		(pts
 			(xy 121.92 128.27) (xy 121.92 130.81)
 		)
@@
 	(wire
 		(pts
+			(xy 78.74 262.89) (xy 83.82 262.89)
+		)
+		(stroke
+			(width 0)
+			(type default)
+		)
+	)
+	(wire
+		(pts
 			(xy 353.06 151.13) (xy 353.06 153.67)
 		)
@@
 	(wire
 		(pts
+			(xy 59.69 265.43) (xy 63.5 265.43)
+		)
+		(stroke
+			(width 0)
+			(type default)
+		)
+	)
+	(wire
+		(pts
 			(xy 335.28 105.41) (xy 335.28 107.95)
 		)
@@
 	(wire
 		(pts
+			(xy 59.69 262.89) (xy 63.5 262.89)
+		)
+		(stroke
+			(width 0)
+			(type default)
+		)
+	)
+	(wire
+		(pts
 			(xy 154.94 82.55) (xy 157.48 82.55)
 		)
@@
 		)
 	)
+	(text "hack to make pads drill correctly\nnot used electrically"
+		(exclude_from_sim no)
+		(at 353.06 54.61 0)
+		(effects
+			(font
+				(size 1.27 1.27)
+			)
+			(justify left)
+		)
+	)
 	(text "Rotary Encoder"
 		(exclude_from_sim no)
@@
 		)
 	)
+	(label "S1"
+		(at 83.82 262.89 180)
+		(effects
+			(font
+				(size 1.27 1.27)
+			)
+			(justify right bottom)
+		)
+	)
+	(label "B"
+		(at 59.69 267.97 0)
+		(effects
+			(font
+				(size 1.27 1.27)
+			)
+			(justify left bottom)
+		)
+	)
+	(label "B"
+		(at 60.96 238.76 0)
+		(effects
+			(font
+				(size 1.27 1.27)
+			)
+			(justify left bottom)
+		)
+	)
+	(label "S1"
+		(at 81.28 233.68 0)
+		(effects
+			(font
+				(size 1.27 1.27)
+			)
+			(justify left bottom)
+		)
+	)
+	(label "A"
+		(at 60.96 233.68 0)
+		(effects
+			(font
+				(size 1.27 1.27)
+			)
+			(justify left bottom)
+		)
+	)
+	(label "SW77"
+		(at 71.12 246.38 0)
+		(effects
+			(font
+				(size 1.27 1.27)
+			)
+			(justify left bottom)
+		)
+	)
+	(label "C"
+		(at 60.96 236.22 0)
+		(effects
+			(font
+				(size 1.27 1.27)
+			)
+			(justify left bottom)
+		)
+	)
+	(label "A"
+		(at 59.69 262.89 0)
+		(effects
+			(font
+				(size 1.27 1.27)
+			)
+			(justify left bottom)
+		)
+	)
+	(label "SW77"
+		(at 360.68 59.69 180)
+		(effects
+			(font
+				(size 1.27 1.27)
+			)
+			(justify right bottom)
+		)
+	)
+	(label "C"
+		(at 59.69 265.43 0)
+		(effects
+			(font
+				(size 1.27 1.27)
+			)
+			(justify left bottom)
+		)
+	)
 	(hierarchical_label "ROW0"
 		(shape input)
@@
 	)
 	(symbol
+		(lib_id "PCM_marbastlib-various:ROT_SKYLOONG_HS-Switch")
+		(at 71.12 265.43 0)
+		(unit 1)
+		(exclude_from_sim no)
+		(in_bom no)
+		(on_board yes)
+		(dnp no)
+		(fields_autoplaced yes)
+		(property "Reference" "SW78"
+			(at 71.12 255.27 0)
+			(effects
+				(font
+					(size 1.27 1.27)
+				)
+			)
+		)
+		(property "Value" "ROT_SKYLOONG_HS"
+			(at 71.12 257.81 0)
+			(effects
+				(font
+					(size 1.27 1.27)
+				)
+			)
+		)
+		(property "Footprint" "PCM_marbastlib-various:ROT_SKYLOONG_HS-Switch"
+			(at 71.12 265.43 0)
+			(effects
+				(font
+					(size 1.27 1.27)
+				)
+				(hide yes)
+			)
+		)
+		(property "Datasheet" "https://skyloong.vip/products/abs-hot-swappable-knobs-madule"
+			(at 71.12 265.43 0)
+			(effects
+				(font
+					(size 1.27 1.27)
+				)
+				(hide yes)
+			)
+		)
+		(property "Description" "SKYLOONG hotswap encoder module"
+			(at 71.12 265.43 0)
+			(effects
+				(font
+					(size 1.27 1.27)
+				)
+				(hide yes)
+			)
+		)
+		(pin "C"
+		)
+		(pin "S"
+		)
+		(pin "B"
+		)
+		(pin "A"
+		)
+		(instances
+			(project ""
+				(path "/9cb56eee-d4d8-48bb-94d9-229fa32a5257/c8b42f60-25dd-4dff-a294-ad95732b9c88"
+					(reference "SW78")
+					(unit 1)
+				)
+			)
+		)
+	)
+	(symbol
 		(lib_id "Device:D")
 		(at 317.5 88.9 270)
@@
 					(unit 1)
 				)
-			)
-		)
-	)
-	(symbol
-		(lib_id "power:GND")
-		(at 71.12 246.38 0)
-		(unit 1)
-		(exclude_from_sim no)
-		(in_bom yes)
-		(on_board yes)
-		(dnp no)
-		(fields_autoplaced yes)
-		(property "Reference" "#PWR012"
-			(at 71.12 252.73 0)
-			(effects
-				(font
-					(size 1.27 1.27)
-				)
-				(hide yes)
-			)
-		)
-		(property "Value" "GND"
-			(at 71.12 251.46 0)
-			(effects
-				(font
-					(size 1.27 1.27)
-				)
-			)
-		)
-		(property "Footprint" ""
-			(at 71.12 246.38 0)
-			(effects
-				(font
-					(size 1.27 1.27)
-				)
-				(hide yes)
-			)
-		)
-		(property "Datasheet" ""
-			(at 71.12 246.38 0)
-			(effects
-				(font
-					(size 1.27 1.27)
-				)
-				(hide yes)
-			)
-		)
-		(property "Description" "Power symbol creates a global label with name \"GND\" , ground"
-			(at 71.12 246.38 0)
-			(effects
-				(font
-					(size 1.27 1.27)
-				)
-				(hide yes)
-			)
-		)
-		(pin "1"
-		)
-		(instances
-			(project "kb"
-				(path "/9cb56eee-d4d8-48bb-94d9-229fa32a5257/c8b42f60-25dd-4dff-a294-ad95732b9c88"
-					(reference "#PWR012")
-					(unit 1)
-				)

Commit message: split backspace
Parts:
- added D77: D, Diode_SMD:D_SOD-123, symbol Device:D
- added SW79: SW_Push, PCM_marbastlib-mx:SW_MX_1u, symbol Switch:SW_Push
Connections:
- net COL13: now also SW45.1
- net COL14: now also SW79.1; no longer SW45.1
- net ROW1: now also D77.1 (K); no longer D30.1 (K)
- net ROW2: now also D30.1 (K)
- new net: D77.2 (A), SW79.2
Other:
- moved on the sheet: D30, D45, SW30, SW45
